Commit message: robot is in rviz and gazebo in playmat and can be controlled by keyboard

File: src/maze/description/inertial_macros.xacro (robot description, xacro)
@@ -12,13 +12,13 @@
     </xacro:macro>
     <!-- Box Inertia Macro -->
-    <xacro:macro name="inertial_box" params="mass x y z">
-        <inertial>
-            <mass value="${mass}"/>
-            <origin xyz="0 0 0" rpy="0 0 0"/>
-            <inertia ixx="${(1/12) * mass * (y * y + z * z)}" ixy="0.0" ixz="0.0"
-                    iyy="${(1/12) * mass * (x * x + z * z)}" iyz="0.0"
-                    izz="${(1/12) * mass * (x * x + y * y)}"/>
-        </inertial>
-    </xacro:macro>
+<xacro:macro name="inertial_box" params="mass x y z origin_xyz:='0 0 0' origin_rpy:='0 0 0'">
+    <inertial>
+        <mass value="${mass}"/>
+        <origin xyz="${origin_xyz}" rpy="${origin_rpy}"/>
+        <inertia ixx="${(1/12) * mass * (y * y + z * z)}" ixy="0.0" ixz="0.0"
+                iyy="${(1/12) * mass * (x * x + z * z)}" iyz="0.0"
+                izz="${(1/12) * mass * (x * x + y * y)}"/>
+    </inertial>
+</xacro:macro>
     <!-- Cylinder Inertia Macro -->
     <xacro:macro name="inertial_cylinder" params="mass length radius">

File: src/maze/description/robot.urdf.xacro (robot description, xacro)
@@ -2,3 +2,4 @@
 <robot xmlns:xacro="http://www.ros.org/wiki/xacro" name="robot">
     <xacro:include filename="robot_core.xacro"/>
+    <xacro:include filename="gazebo_control.xacro"/>
 </robot>

File: src/maze/description/robot_core.xacro (robot description, xacro)
@@ -37,6 +37,9 @@
             </geometry>
         </collision>
-        <xacro:inertial_box mass="0.5" x="0.3" y="0.3" z="0.15"/>
+        <xacro:inertial_box mass="1.0" x="0.3" y="0.3" z="0.15" origin_xyz="0.1 0 -0.05" origin_rpy="0 0 0"/>
     </link>
+    <gazebo reference="chassis">
+        <material>Gazebo/White</material>
+    </gazebo>
     <!-- Left Wheel -->
     <joint name="left_wheel_joint" type="continuous">
@@ -60,4 +63,7 @@
         <xacro:inertial_cylinder mass="0.1" length="0.03" radius="0.0342"/>
     </link>
+    <gazebo reference="left_wheel">
+        <material>Gazebo/Blue</material>
+    </gazebo>
     <!-- Right Wheel -->
     <joint name="right_wheel_joint" type="continuous">
@@ -81,4 +87,7 @@
         <xacro:inertial_cylinder mass="0.1" length="0.03" radius="0.0342"/>
     </link>
+    <gazebo reference="right_wheel">
+        <material>Gazebo/Blue</material>
+    </gazebo>
     <!-- Caster Wheel -->
     <joint name="caster_wheel_joint" type="fixed">
@@ -101,3 +110,8 @@
         <xacro:inertial_sphere mass="0.1" radius="0.0342"/>
     </link>
+    <gazebo reference="caster_wheel">
+        <material>Gazebo/Black</material>
+        <mu1 value="0.0001"/>
+        <mu2 value="0.0001"/>
+    </gazebo>
 </robot>
