Commit message: should be working but controlmanager is not and /opt/ros/humble/share/gazebo_ros2_control/gazebo_ros2_control_plugins.xml is missing

File: install/robonav/share/robonav/description/inertial_macros.xacro (robot description, xacro)
@@ -1 +1 @@
-/home/ferdinand/2024-2025-Robotics-cup/src/maze/description/inertial_macros.xacro
+/home/ferdinand/2024-2025-Robotics-cup/src/robonav/description/inertial_macros.xacro

File: install/robonav/share/robonav/description/robot.urdf.xacro (robot description, xacro)
@@ -1 +1 @@
-/home/ferdinand/2024-2025-Robotics-cup/src/maze/description/robot.urdf.xacro
+/home/ferdinand/2024-2025-Robotics-cup/src/robonav/description/robot.urdf.xacro

File: install/robonav/share/robonav/description/robot_core.xacro (robot description, xacro)
@@ -1 +1 @@
-/home/ferdinand/2024-2025-Robotics-cup/src/maze/description/robot_core.xacro
+/home/ferdinand/2024-2025-Robotics-cup/src/robonav/description/robot_core.xacro

File: src/robonav/description/robot_core.xacro (robot description, xacro)
@@ -115,3 +115,44 @@
         <mu2 value="0.0001"/>
     </gazebo>
+    <ros2_control name="DiffDriveController" type="system">
+        <hardware>
+            <plugin>gazebo_ros2_control/GazeboSystem</plugin>
+        </hardware>
+        <joint name="left_wheel_joint">
+            <command_interface name="velocity"/>
+            <state_interface name="position"/>
+            <state_interface name="velocity"/>
+        </joint>
+        <joint name="right_wheel_joint">
+            <command_interface name="velocity"/>
+            <state_interface name="position"/>
+            <state_interface name="velocity"/>
+        </joint>
+    </ros2_control>
+    <gazebo>
+        <plugin filename="libgazebo_ros2_control.so" name="gazebo_ros2_control">
+            <robotSimType>gazebo_ros2_control/GazeboSystem</robotSimType>
+        </plugin>
+    </gazebo>
+    <!-- <ros2_control name="GazeboSystem" type="system">
+        <hardware>
+            <plugin>libgazebo_ros2_control/GazeboSystem</plugin>
+        </hardware>
+        <joint name="left_wheel_joint">
+        <command_interface name="velocity">
+            <param name="min">-1</param>
+            <param name="max">1</param>
+        </command_interface>
+        <state_interface name="position"/>
+        <state_interface name="velocity"/>
+        </joint>
+        <joint name="right_wheel_joint">
+        <command_interface name="velocity">
+            <param name="min">-1</param>
+            <param name="max">1</param>
+        </command_interface>
+        <state_interface name="position"/>
+        <state_interface name="velocity"/>
+        </joint>
+    </ros2_control> -->
 </robot>

Commit message: robot moving

File: install/robonav/share/robonav/description/inertial_macros.xacro (robot description, xacro)
@@ -1 +1,33 @@
-/home/ferdinand/2024-2025-Robotics-cup/src/maze/description/inertial_macros.xacro
+<?xml version="1.0"?>
+<robot xmlns:xacro="http://www.ros.org/wiki/xacro">
+    <!-- Sphere Inertia Macro -->
+    <xacro:macro name="inertial_sphere" params="mass radius">
+        <inertial>
+            <mass value="${mass}"/>
+            <origin xyz="0 0 0" rpy="0 0 0"/>
+            <inertia ixx="${(2/5) * mass * (radius * radius)}" ixy="0.0" ixz="0.0"
+                    iyy="${(2/5) * mass * (radius * radius)}" iyz="0.0"
+                    izz="${(2/5) * mass * (radius * radius)}"/>
+        </inertial>
+    </xacro:macro>
+    <!-- Box Inertia Macro -->
+<xacro:macro name="inertial_box" params="mass x y z origin_xyz:='0 0 0' origin_rpy:='0 0 0'">
+    <inertial>
+        <mass value="${mass}"/>
+        <origin xyz="${origin_xyz}" rpy="${origin_rpy}"/>
+        <inertia ixx="${(1/12) * mass * (y * y + z * z)}" ixy="0.0" ixz="0.0"
+                iyy="${(1/12) * mass * (x * x + z * z)}" iyz="0.0"
+                izz="${(1/12) * mass * (x * x + y * y)}"/>
+    </inertial>
+</xacro:macro>
+    <!-- Cylinder Inertia Macro -->
+    <xacro:macro name="inertial_cylinder" params="mass length radius">
+        <inertial>
+            <mass value="${mass}"/>
+            <origin xyz="0 0 0" rpy="0 0 0"/>
+            <inertia ixx="${(1/12) * mass * (3 * radius * radius + length * length)}" ixy="0.0" ixz="0.0"
+                    iyy="${(1/12) * mass * (3 * radius * radius + length * length)}" iyz="0.0"
+                    izz="${(1/2) * mass * (radius * radius)}"/>
+        </inertial>
+    </xacro:macro>
+</robot>

File: install/robonav/share/robonav/description/robot.urdf.xacro (robot description, xacro)
@@ -1 +1,5 @@
-/home/ferdinand/2024-2025-Robotics-cup/src/maze/description/robot.urdf.xacro
+<?xml version="1.0"?>
+<robot xmlns:xacro="http://www.ros.org/wiki/xacro" name="robot">
+    <xacro:include filename="robot_core.xacro"/>
+    <xacro:include filename="gazebo_control.xacro"/>
+</robot>

File: install/robonav/share/robonav/description/robot_core.xacro (robot description, xacro)
@@ -1 +1,117 @@
-/home/ferdinand/2024-2025-Robotics-cup/src/maze/description/robot_core.xacro
+<?xml version="1.0"?>
+<robot xmlns:xacro="http://www.ros.org/wiki/xacro">
+    <xacro:include filename="inertial_macros.xacro"/>
+    <!-- Define Colors -->
+    <material name="white">
+        <color rgba="1 1 1 1"/>
+    </material>
+    <material name="orange">
+        <color rgba="1 0.3 0.1 1"/>
+    </material>
+    <material name="blue">
+        <color rgba="0.2 0.2 1 1"/>
+    </material>
+    <material name="black">
+        <color rgba="0 0 0 1"/>
+    </material>
+    <!-- Base Link -->
+    <link name="base_link"/>
+    <!-- Chassis -->
+    <joint name="chassis_joint" type="fixed">
+        <parent link="base_link"/>
+        <child link="chassis"/>
+        <origin xyz="-0.1 0 0"/>
+    </joint>
+    <link name="chassis">
+        <visual>
+            <origin xyz="0.15 0 0.075" rpy="0 0 0"/>
+            <geometry>
+                <box size="0.3 0.3 0.15"/>
+            </geometry>
+            <material name="white"/>
+        </visual>
+        <collision>
+            <origin xyz="0.15 0 0.075" rpy="0 0 0"/>
+            <geometry>
+                <box size="0.3 0.3 0.15"/>
+            </geometry>
+        </collision>
+        <xacro:inertial_box mass="1.0" x="0.3" y="0.3" z="0.15" origin_xyz="0.1 0 -0.05" origin_rpy="0 0 0"/>
+    </link>
+    <gazebo reference="chassis">
+        <material>Gazebo/White</material>
+    </gazebo>
+    <!-- Left Wheel -->
+    <joint name="left_wheel_joint" type="continuous">
+        <parent link="base_link"/>
+        <child link="left_wheel"/>
+        <origin xyz="0 0.175 0" rpy="-${pi/2} 0 0"/>
+        <axis xyz="0 0 1"/>
+    </joint>
+    <link name="left_wheel">
+        <visual>
+            <geometry>
+                <cylinder radius="0.0342" length="0.03"/>
+            </geometry>
+            <material name="blue"/>
+        </visual>
+        <collision>
+            <geometry>
+                <cylinder radius="0.0342" length="0.03"/>
+            </geometry>
+        </collision>
+        <xacro:inertial_cylinder mass="0.1" length="0.03" radius="0.0342"/>
+    </link>
+    <gazebo reference="left_wheel">
+        <material>Gazebo/Blue</material>
+    </gazebo>
+    <!-- Right Wheel -->
+    <joint name="right_wheel_joint" type="continuous">
+        <parent link="base_link"/>
+        <child link="right_wheel"/>
+        <origin xyz="0 -0.175 0" rpy="${pi/2} 0 0"/>
+        <axis xyz="0 0 -1"/>
+    </joint>
+    <link name="right_wheel">
+        <visual>
+            <geometry>
+                <cylinder radius="0.0342" length="0.03"/>
+            </geometry>
+            <material name="blue"/>
+        </visual>
+        <collision>
+            <geometry>
+                <cylinder radius="0.0342" length="0.03"/>
+            </geometry>
+        </collision>
+        <xacro:inertial_cylinder mass="0.1" length="0.03" radius="0.0342"/>
+    </link>
+    <gazebo reference="right_wheel">
+        <material>Gazebo/Blue</material>
+    </gazebo>
+    <!-- Caster Wheel -->
+    <joint name="caster_wheel_joint" type="fixed">
+        <parent link="chassis"/>
+        <child link="caster_wheel"/>
+        <origin xyz="0.24 0 0" rpy="0 0 0"/>
+    </joint>
+    <link name="caster_wheel">
+        <visual>
+            <geometry>
+                <sphere radius="0.0342"/>
+            </geometry>
+            <material name="black"/>
+        </visual>
+        <collision>
+            <geometry>
+                <sphere radius="0.0342"/>
+            </geometry>
+        </collision>
+        <xacro:inertial_sphere mass="0.1" radius="0.0342"/>
+    </link>
+    <gazebo reference="caster_wheel">
+        <material>Gazebo/Black</material>
+        <mu1 value="0.0001"/>
+        <mu2 value="0.0001"/>
+    </gazebo>
+</robot>
