Commit message: removed dt, dt = real execution time, improved some things, but still different in gazbeo

File: src/robonav/description/gazebo_control.xacro (robot description, xacro)
@@ -6,5 +6,5 @@
             <left_joint>left_wheel_joint</left_joint>
             <right_joint>right_wheel_joint</right_joint>
-            <wheel_separation>0.35</wheel_separation>
+            <wheel_separation>0.33</wheel_separation>
             <wheel_diameter>0.0432</wheel_diameter>
             <!-- Limits -->
@@ -17,4 +17,6 @@
             <publish_odom_tf>true</publish_odom_tf>
             <publish_wheel_tf>true</publish_wheel_tf>
+            <!-- Update Rate -->
+            <update_rate>50.0</update_rate>
         </plugin>
     </gazebo>

File: src/robonav/description/robot_core.xacro (robot description, xacro)
@@ -46,5 +46,5 @@
         <parent link="base_link"/>
         <child link="left_wheel"/>
-        <origin xyz="0 0.175 0" rpy="-${pi/2} 0 0"/>
+        <origin xyz="0 0.15 0" rpy="-${pi/2} 0 0"/>
         <axis xyz="0 0 1"/>
     </joint>
@@ -70,5 +70,5 @@
         <parent link="base_link"/>
         <child link="right_wheel"/>
-        <origin xyz="0 -0.175 0" rpy="${pi/2} 0 0"/>
+        <origin xyz="0 -0.15 0" rpy="${pi/2} 0 0"/>
         <axis xyz="0 0 -1"/>
     </joint>
@@ -115,3 +115,23 @@
         <mu2 value="0.0001"/>
     </gazebo>
+    <transmission name="left_wheel_joint_tran">
+        <type>transmission_interface/SimpleTransmission</type>
+        <joint name="left_wheel_joint">
+            <hardwareInterface>hardware_interface/EffortJointInterface</hardwareInterface>
+        </joint>
+        <actuator name="left_wheel_joint_actr">
+            <hardwareInterface>hardware_interface/EffortJointInterface</hardwareInterface>
+            <mechanicalReduction>1</mechanicalReduction>
+        </actuator>
+    </transmission>
+        <transmission name="right_wheel_joint_tran">
+        <type>transmission_interface/SimpleTransmission</type>
+        <joint name="right_wheel_joint">
+            <hardwareInterface>hardware_interface/EffortJointInterface</hardwareInterface>
+        </joint>
+        <actuator name="right_wheel_joint_actr">
+            <hardwareInterface>hardware_interface/EffortJointInterface</hardwareInterface>
+            <mechanicalReduction>1</mechanicalReduction>
+        </actuator>
+    </transmission>
 </robot>

Commit message: added AMCL and laser to pointcloud2 but not yet tuned

File: src/robonav/description/gazebo_control.xacro (robot description, xacro)
@@ -13,5 +13,5 @@
             <!-- Output -->
             <odometry_frame>odom</odometry_frame>
-            <robot_base_frame>base_link</robot_base_frame>
+            <robot_base_frame>base_footprint</robot_base_frame>
             <publish_odom>true</publish_odom>
             <publish_odom_tf>true</publish_odom_tf>

File: src/robonav/description/robot_core.xacro (robot description, xacro)
@@ -15,4 +15,11 @@
         <color rgba="0 0 0 1"/>
     </material>
+    <!-- Base Footprint -->
+    <link name="base_footprint"/>
+    <joint name="base_footprint_joint" type="fixed">
+        <parent link="base_footprint"/>
+        <child link="base_link"/>
+        <origin xyz="0 0 0" rpy="0 0 0"/>
+    </joint>
     <!-- Base Link -->
     <link name="base_link"/>

File: src/robonav/description/rplidar_c1.xacro (robot description, xacro)
@@ -26,5 +26,5 @@
     <!-- Joint Lidar to Robot (chassis) -->
     <joint name="rplidar_joint" type="fixed">
-        <parent link="chassis"/>
+        <parent link="base_link"/>
         <child link="lidar_link"/>
         <origin xyz="0.12 0.0 0.35" rpy="0 0 0"/>  <!-- Lidar is on top of the Chassis -->

Commit message: added big robot, removed base_footprint, smoothing for obstacle...

File: src/robonav/description/gazebo_control.xacro (robot description, xacro)
@@ -13,5 +13,5 @@
             <!-- Output -->
             <odometry_frame>odom</odometry_frame>
-            <robot_base_frame>base_footprint</robot_base_frame>
+            <robot_base_frame>base_link</robot_base_frame>
             <publish_odom>true</publish_odom>
             <publish_odom_tf>true</publish_odom_tf>

File: src/robonav/description/robot_core_small.xacro (robot description, xacro)
@@ -15,11 +15,11 @@
         <color rgba="0 0 0 1"/>
     </material>
-    <!-- Base Footprint
+    <!-- Base Footprint -->
     <link name="base_footprint"/>
     <joint name="base_footprint_joint" type="fixed">
         <parent link="base_footprint"/>
         <child link="base_link"/>
-        <origin xyz="0 0 0.044" rpy="0 0 0"/>
-    </joint> -->
+        <origin xyz="0 0 0" rpy="0 0 0"/>
+    </joint>
     <!-- Base Link -->
     <link name="base_link"/>
@@ -30,30 +30,28 @@
         <origin xyz="-0.1 0 0"/>
     </joint>
-    <!-- xyz = 172 of box dimesions, x is forward, y is to the sides -->
     <link name="chassis">
         <visual>
-            <origin xyz="0.1775 0 0.175" rpy="0 0 0"/>
+            <origin xyz="0.15 0 0.075" rpy="0 0 0"/>
             <geometry>
-                <box size="0.4 0.355 0.350"/>
+                <box size="0.25 0.25 0.15"/>
             </geometry>
             <material name="white"/>
         </visual>
         <collision>
-            <origin xyz="0.1775 0 0.175" rpy="0 0 0"/>
+            <origin xyz="0.15 0 0.075" rpy="0 0 0"/>
             <geometry>
-                <box size="0.4 0.355 0.350"/>
+                <box size="0.25 0.25 0.15"/>
             </geometry>
         </collision>
-        <xacro:inertial_box mass="1.0" x="0.355" y="0.400" z="0.350" origin_xyz="0.1 0 -0.05" origin_rpy="0 0 0"/>
+        <xacro:inertial_box mass="1.0" x="0.25" y="0.25" z="0.15" origin_xyz="0.1 0 -0.05" origin_rpy="0 0 0"/>
     </link>
     <gazebo reference="chassis">
         <material>Gazebo/White</material>
     </gazebo>
-    <!-- TRACK WIDTH: 373 -->
     <!-- Left Wheel -->
     <joint name="left_wheel_joint" type="continuous">
         <parent link="base_link"/>
         <child link="left_wheel"/>
-        <origin xyz="0 0.1865 0" rpy="-${pi/2} 0 0"/>
+        <origin xyz="0 0.15 0" rpy="-${pi/2} 0 0"/>
         <axis xyz="0 0 1"/>
     </joint>
@@ -61,5 +59,5 @@
         <visual>
             <geometry>
-                <cylinder radius="0.044" length="0.01"/>
+                <cylinder radius="0.0342" length="0.03"/>
             </geometry>
             <material name="blue"/>
@@ -67,8 +65,8 @@
         <collision>
             <geometry>
-                <cylinder radius="0.044" length="0.01"/>
+                <cylinder radius="0.0342" length="0.03"/>
             </geometry>
         </collision>
-        <xacro:inertial_cylinder mass="0.1" length="0.01" radius="0.044"/>
+        <xacro:inertial_cylinder mass="0.1" length="0.03" radius="0.0342"/>
     </link>
     <gazebo reference="left_wheel">
@@ -79,5 +77,5 @@
         <parent link="base_link"/>
         <child link="right_wheel"/>
-        <origin xyz="0 -0.1865 0" rpy="${pi/2} 0 0"/>
+        <origin xyz="0 -0.15 0" rpy="${pi/2} 0 0"/>
         <axis xyz="0 0 -1"/>
     </joint>
@@ -85,5 +83,5 @@
         <visual>
             <geometry>
-                <cylinder radius="0.044" length="0.01"/>
+                <cylinder radius="0.0342" length="0.03"/>
             </geometry>
             <material name="blue"/>
@@ -91,8 +89,8 @@
         <collision>
             <geometry>
-                <cylinder radius="0.044" length="0.01"/>
+                <cylinder radius="0.0342" length="0.03"/>
             </geometry>
         </collision>
-        <xacro:inertial_cylinder mass="0.1" length="0.01" radius="0.044"/>
+        <xacro:inertial_cylinder mass="0.1" length="0.03" radius="0.0342"/>
     </link>
     <gazebo reference="right_wheel">
@@ -103,10 +101,10 @@
         <parent link="chassis"/>
         <child link="caster_wheel"/>
-        <origin xyz="0.3 0 0" rpy="0 0 0"/>
+        <origin xyz="0.24 0 0" rpy="0 0 0"/>
     </joint>
     <link name="caster_wheel">
         <visual>
             <geometry>
-                <sphere radius="0.044"/>
+                <sphere radius="0.0342"/>
             </geometry>
             <material name="black"/>
@@ -114,16 +112,8 @@
         <collision>
             <geometry>
-                <sphere radius="0.044"/>
+                <sphere radius="0.0342"/>
             </geometry>
-            <surface>
-                <friction>
-                    <ode>
-                        <mu>0.08</mu>
-                        <mu2>0.08</mu2>
-                    </ode>
-                </friction>
-            </surface>
         </collision>
-        <xacro:inertial_sphere mass="0.1" radius="0.044"/>
+        <xacro:inertial_sphere mass="0.1" radius="0.0342"/>
     </link>
     <gazebo reference="caster_wheel">

File: src/robonav/description/rplidar_c1.xacro (robot description, xacro)
@@ -28,5 +28,5 @@
         <parent link="base_link"/>
         <child link="lidar_link"/>
-        <origin xyz="0.12 0.0 0.35" rpy="0 0 0"/>  <!-- Lidar is on top of the Chassis -->
+        <origin xyz="0.1 0.0 0.365" rpy="0 0 0"/>  <!-- Lidar is on top of the Chassis -->
     </joint>
     <!-- Lidar Plugin -->
