Commit message: robot pathfollowing and simple world gazebo, path in rviz

File: src/robonav/description/robot_core.xacro (robot description, xacro)
@@ -7,5 +7,5 @@
     </material>
     <material name="orange">
-        <color rgba="1 0.3 0.1 1"/>
+        <color rgba="1 0.25 0.1 1"/>
     </material>
     <material name="blue">
@@ -27,5 +27,5 @@
             <origin xyz="0.15 0 0.075" rpy="0 0 0"/>
             <geometry>
-                <box size="0.3 0.3 0.15"/>
+                <box size="0.25 0.25 0.15"/>
             </geometry>
             <material name="white"/>
@@ -34,8 +34,8 @@
             <origin xyz="0.15 0 0.075" rpy="0 0 0"/>
             <geometry>
-                <box size="0.3 0.3 0.15"/>
+                <box size="0.25 0.25 0.15"/>
             </geometry>
         </collision>
-        <xacro:inertial_box mass="1.0" x="0.3" y="0.3" z="0.15" origin_xyz="0.1 0 -0.05" origin_rpy="0 0 0"/>
+        <xacro:inertial_box mass="1.0" x="0.25" y="0.25" z="0.15" origin_xyz="0.1 0 -0.05" origin_rpy="0 0 0"/>
     </link>
     <gazebo reference="chassis">

Commit message: working fine exept path sending and PID

File: src/robonav/description/robot_core.xacro (robot description, xacro)
@@ -14,5 +14,5 @@
             <origin xyz="0.15 0 0.075" rpy="0 0 0"/>
             <geometry>
-                <box size="0.25 0.25 0.15"/>
+                <box size="0.25 0.18 0.15"/>
             </geometry>
             <material name="blue">
@@ -23,5 +23,5 @@
             <origin xyz="0.15 0 0.075" rpy="0 0 0"/>
             <geometry>
-                <box size="0.25 0.25 0.15"/>
+                <box size="0.25 0.18 0.15"/>
             </geometry>
         </collision>
@@ -32,5 +32,5 @@
         <parent link="base_link"/>
         <child link="left_wheel"/>
-        <origin xyz="0 0.15 0" rpy="-${pi/2} 0 0"/>
+        <origin xyz="0 0.0925 0" rpy="-${pi/2} 0 0"/>
         <axis xyz="0 0 1"/>
     </joint>
@@ -55,5 +55,5 @@
         <parent link="base_link"/>
         <child link="right_wheel"/>
-        <origin xyz="0 -0.15 0" rpy="${pi/2} 0 0"/>
+        <origin xyz="0 -0.0925 0" rpy="${pi/2} 0 0"/>
         <axis xyz="0 0 -1"/>
     </joint>

Commit message: Path following and communication with RPI and RSP working! Also vizualization in RVIZ

File: src/robonav/description/robot_core.xacro (robot description, xacro)
@@ -16,6 +16,6 @@
                 <box size="0.25 0.18 0.15"/>
             </geometry>
-            <material name="blue">
-                <color rgba="0.0 0.0 1.0 1.0"/>
+            <material name="light_blue">
+                <color rgba="0.5 0.5 1.0 1.0"/>
             </material>
         </visual>
@@ -40,6 +40,6 @@
                 <cylinder radius="0.0342" length="0.03"/>
             </geometry>
-            <material name="black">
-                <color rgba="0.0 0.0 0.0 1.0"/>
+            <material name="gray">
+                <color rgba="0.5 0.5 0.5 1.0"/>
             </material>
         </visual>
@@ -63,6 +63,6 @@
                 <cylinder radius="0.0342" length="0.03"/>
             </geometry>
-            <material name="black">
-                <color rgba="0.0 0.0 0.0 1.0"/>
+            <material name="gray">
+                <color rgba="0.5 0.5 0.5 1.0"/>
             </material>
         </visual>
@@ -85,6 +85,6 @@
                 <sphere radius="0.0342"/>
             </geometry>
-            <material name="black">
-                <color rgba="0.0 0.0 0.0 1.0"/>
+            <material name="gray">
+                <color rgba="0.5 0.5 0.5 1.0"/>
             </material>
         </visual>

Commit message: added big robot and tuned pid and settings

File: src/robonav/description/robot_core.xacro (robot description, xacro)
@@ -2,4 +2,24 @@
 <robot xmlns:xacro="http://www.ros.org/wiki/xacro">
     <xacro:include filename="inertial_macros.xacro"/>
+    <!-- Define Colors -->
+    <material name="white">
+        <color rgba="1 1 1 1"/>
+    </material>
+    <material name="orange">
+        <color rgba="1 0.25 0.1 1"/>
+    </material>
+    <material name="blue">
+        <color rgba="0.2 0.2 1 1"/>
+    </material>
+    <material name="black">
+        <color rgba="0 0 0 1"/>
+    </material>
+    <!-- Base Footprint
+    <link name="base_footprint"/>
+    <joint name="base_footprint_joint" type="fixed">
+        <parent link="base_footprint"/>
+        <child link="base_link"/>
+        <origin xyz="0 0 0.044" rpy="0 0 0"/>
+    </joint> -->
     <!-- Base Link -->
     <link name="base_link"/>
@@ -10,27 +30,30 @@
         <origin xyz="-0.1 0 0"/>
     </joint>
+    <!-- xyz = 172 of box dimesions, x is forward, y is to the sides -->
     <link name="chassis">
         <visual>
-            <origin xyz="0.15 0 0.075" rpy="0 0 0"/>
+            <origin xyz="0.1775 0 0.175" rpy="0 0 0"/>
             <geometry>
-                <box size="0.25 0.18 0.15"/>
+                <box size="0.4 0.355 0.350"/>
             </geometry>
-            <material name="light_blue">
-                <color rgba="0.5 0.5 1.0 1.0"/>
-            </material>
+            <material name="white"/>
         </visual>
         <collision>
-            <origin xyz="0.15 0 0.075" rpy="0 0 0"/>
+            <origin xyz="0.1775 0 0.175" rpy="0 0 0"/>
             <geometry>
-                <box size="0.25 0.18 0.15"/>
+                <box size="0.4 0.355 0.350"/>
             </geometry>
         </collision>
-        <xacro:inertial_box mass="1.0" x="0.25" y="0.25" z="0.15" origin_xyz="0.1 0 -0.05" origin_rpy="0 0 0"/>
+        <xacro:inertial_box mass="1.0" x="0.355" y="0.400" z="0.350" origin_xyz="0.1 0 -0.05" origin_rpy="0 0 0"/>
     </link>
+    <gazebo reference="chassis">
+        <material>Gazebo/White</material>
+    </gazebo>
+    <!-- TRACK WIDTH: 373 -->
     <!-- Left Wheel -->
     <joint name="left_wheel_joint" type="fixed">
         <parent link="base_link"/>
         <child link="left_wheel"/>
-        <origin xyz="0 0.0925 0" rpy="-${pi/2} 0 0"/>
+        <origin xyz="0 0.1865 0" rpy="-${pi/2} 0 0"/>
         <axis xyz="0 0 1"/>
     </joint>
@@ -38,22 +61,23 @@
         <visual>
             <geometry>
-                <cylinder radius="0.0342" length="0.03"/>
+                <cylinder radius="0.044" length="0.01"/>
             </geometry>
-            <material name="gray">
-                <color rgba="0.5 0.5 0.5 1.0"/>
-            </material>
+            <material name="blue"/>
         </visual>
         <collision>
             <geometry>
-                <cylinder radius="0.0342" length="0.03"/>
+                <cylinder radius="0.044" length="0.01"/>
             </geometry>
         </collision>
-        <xacro:inertial_cylinder mass="0.1" length="0.03" radius="0.0342"/>
+        <xacro:inertial_cylinder mass="0.1" length="0.01" radius="0.044"/>
     </link>
+    <gazebo reference="left_wheel">
+        <material>Gazebo/Blue</material>
+    </gazebo>
     <!-- Right Wheel -->
     <joint name="right_wheel_joint" type="fixed">
         <parent link="base_link"/>
         <child link="right_wheel"/>
-        <origin xyz="0 -0.0925 0" rpy="${pi/2} 0 0"/>
+        <origin xyz="0 -0.1865 0" rpy="${pi/2} 0 0"/>
         <axis xyz="0 0 -1"/>
     </joint>
@@ -61,38 +85,70 @@
         <visual>
             <geometry>
-                <cylinder radius="0.0342" length="0.03"/>
+                <cylinder radius="0.044" length="0.01"/>
             </geometry>
-            <material name="gray">
-                <color rgba="0.5 0.5 0.5 1.0"/>
-            </material>
+            <material name="blue"/>
         </visual>
         <collision>
             <geometry>
-                <cylinder radius="0.0342" length="0.03"/>
+                <cylinder radius="0.044" length="0.01"/>
             </geometry>
         </collision>
-        <xacro:inertial_cylinder mass="0.1" length="0.03" radius="0.0342"/>
+        <xacro:inertial_cylinder mass="0.1" length="0.01" radius="0.044"/>
     </link>
+    <gazebo reference="right_wheel">
+        <material>Gazebo/Blue</material>
+    </gazebo>
     <!-- Caster Wheel -->
     <joint name="caster_wheel_joint" type="fixed">
         <parent link="chassis"/>
         <child link="caster_wheel"/>
-        <origin xyz="0.24 0 0" rpy="0 0 0"/>
+        <origin xyz="0.3 0 0" rpy="0 0 0"/>
     </joint>
     <link name="caster_wheel">
         <visual>
             <geometry>
-                <sphere radius="0.0342"/>
+                <sphere radius="0.044"/>
             </geometry>
-            <material name="gray">
-                <color rgba="0.5 0.5 0.5 1.0"/>
-            </material>
+            <material name="black"/>
         </visual>
         <collision>
             <geometry>
-                <sphere radius="0.0342"/>
+                <sphere radius="0.044"/>
             </geometry>
+            <surface>
+                <friction>
+                    <ode>
+                        <mu>0.08</mu>
+                        <mu2>0.08</mu2>
+                    </ode>
+                </friction>
+            </surface>
         </collision>
-        <xacro:inertial_sphere mass="0.1" radius="0.0342"/>
+        <xacro:inertial_sphere mass="0.1" radius="0.044"/>
     </link>
+    <gazebo reference="caster_wheel">
+        <material>Gazebo/Black</material>
+        <mu1 value="0.0001"/>
+        <mu2 value="0.0001"/>
+    </gazebo>
+    <transmission name="left_wheel_joint_tran">
+        <type>transmission_interface/SimpleTransmission</type>
+        <joint name="left_wheel_joint">
+            <hardwareInterface>hardware_interface/EffortJointInterface</hardwareInterface>
+        </joint>
+        <actuator name="left_wheel_joint_actr">
+            <hardwareInterface>hardware_interface/EffortJointInterface</hardwareInterface>
+            <mechanicalReduction>1</mechanicalReduction>
+        </actuator>
+    </transmission>
+        <transmission name="right_wheel_joint_tran">
+        <type>transmission_interface/SimpleTransmission</type>
+        <joint name="right_wheel_joint">
+            <hardwareInterface>hardware_interface/EffortJointInterface</hardwareInterface>
+        </joint>
+        <actuator name="right_wheel_joint_actr">
+            <hardwareInterface>hardware_interface/EffortJointInterface</hardwareInterface>
+            <mechanicalReduction>1</mechanicalReduction>
+        </actuator>
+    </transmission>
 </robot>
