Commit message: rviz vizualization, but robot model not moving and robot moving weird, path sending is taking long

File: src/robonav/description/robot.urdf.xacro (robot description, xacro)
@@ -2,4 +2,3 @@
 <robot xmlns:xacro="http://www.ros.org/wiki/xacro" name="robot">
     <xacro:include filename="robot_core.xacro"/>
-    <xacro:include filename="gazebo_control.xacro"/>
 </robot>

File: src/robonav/description/robot_core.xacro (robot description, xacro)
@@ -2,17 +2,4 @@
 <robot xmlns:xacro="http://www.ros.org/wiki/xacro">
     <xacro:include filename="inertial_macros.xacro"/>
-    <!-- Define Colors -->
-    <material name="white">
-        <color rgba="1 1 1 1"/>
-    </material>
-    <material name="orange">
-        <color rgba="1 0.25 0.1 1"/>
-    </material>
-    <material name="blue">
-        <color rgba="0.2 0.2 1 1"/>
-    </material>
-    <material name="black">
-        <color rgba="0 0 0 1"/>
-    </material>
     <!-- Base Link -->
     <link name="base_link"/>
@@ -29,5 +16,7 @@
                 <box size="0.25 0.25 0.15"/>
             </geometry>
-            <material name="white"/>
+            <material name="blue">
+                <color rgba="0.0 0.0 1.0 1.0"/>
+            </material>
         </visual>
         <collision>
@@ -39,9 +28,6 @@
         <xacro:inertial_box mass="1.0" x="0.25" y="0.25" z="0.15" origin_xyz="0.1 0 -0.05" origin_rpy="0 0 0"/>
     </link>
-    <gazebo reference="chassis">
-        <material>Gazebo/White</material>
-    </gazebo>
     <!-- Left Wheel -->
-    <joint name="left_wheel_joint" type="continuous">
+    <joint name="left_wheel_joint" type="fixed">
         <parent link="base_link"/>
         <child link="left_wheel"/>
@@ -54,5 +40,7 @@
                 <cylinder radius="0.0342" length="0.03"/>
             </geometry>
-            <material name="blue"/>
+            <material name="black">
+                <color rgba="0.0 0.0 0.0 1.0"/>
+            </material>
         </visual>
         <collision>
@@ -63,9 +51,6 @@
         <xacro:inertial_cylinder mass="0.1" length="0.03" radius="0.0342"/>
     </link>
-    <gazebo reference="left_wheel">
-        <material>Gazebo/Blue</material>
-    </gazebo>
     <!-- Right Wheel -->
-    <joint name="right_wheel_joint" type="continuous">
+    <joint name="right_wheel_joint" type="fixed">
         <parent link="base_link"/>
         <child link="right_wheel"/>
@@ -78,5 +63,7 @@
                 <cylinder radius="0.0342" length="0.03"/>
             </geometry>
-            <material name="blue"/>
+            <material name="black">
+                <color rgba="0.0 0.0 0.0 1.0"/>
+            </material>
         </visual>
         <collision>
@@ -87,7 +74,4 @@
         <xacro:inertial_cylinder mass="0.1" length="0.03" radius="0.0342"/>
     </link>
-    <gazebo reference="right_wheel">
-        <material>Gazebo/Blue</material>
-    </gazebo>
     <!-- Caster Wheel -->
     <joint name="caster_wheel_joint" type="fixed">
@@ -101,5 +85,7 @@
                 <sphere radius="0.0342"/>
             </geometry>
-            <material name="black"/>
+            <material name="black">
+                <color rgba="0.0 0.0 0.0 1.0"/>
+            </material>
         </visual>
         <collision>
@@ -110,28 +96,3 @@
         <xacro:inertial_sphere mass="0.1" radius="0.0342"/>
     </link>
-    <gazebo reference="caster_wheel">
-        <material>Gazebo/Black</material>
-        <mu1 value="0.0001"/>
-        <mu2 value="0.0001"/>
-    </gazebo>
-    <transmission name="left_wheel_joint_tran">
-        <type>transmission_interface/SimpleTransmission</type>
-        <joint name="left_wheel_joint">
-            <hardwareInterface>hardware_interface/EffortJointInterface</hardwareInterface>
-        </joint>
-        <actuator name="left_wheel_joint_actr">
-            <hardwareInterface>hardware_interface/EffortJointInterface</hardwareInterface>
-            <mechanicalReduction>1</mechanicalReduction>
-        </actuator>
-    </transmission>
-        <transmission name="right_wheel_joint_tran">
-        <type>transmission_interface/SimpleTransmission</type>
-        <joint name="right_wheel_joint">
-            <hardwareInterface>hardware_interface/EffortJointInterface</hardwareInterface>
-        </joint>
-        <actuator name="right_wheel_joint_actr">
-            <hardwareInterface>hardware_interface/EffortJointInterface</hardwareInterface>
-            <mechanicalReduction>1</mechanicalReduction>
-        </actuator>
-    </transmission>
 </robot>

Commit message: changrd wheel distance to 37,6mm and made robot model good for rviz

File: src/robonav/description/robot.urdf.xacro (robot description, xacro)
@@ -1,4 +1,5 @@
 <?xml version="1.0"?>
 <robot xmlns:xacro="http://www.ros.org/wiki/xacro" name="robot">
+    <xacro:include filename="materials.xacro"/>
     <xacro:include filename="robot_core.xacro"/>
     <xacro:include filename="rplidar_c1.xacro"/>

File: src/robonav/description/robot_core.xacro (robot description, xacro)
@@ -2,17 +2,5 @@
 <robot xmlns:xacro="http://www.ros.org/wiki/xacro">
     <xacro:include filename="inertial_macros.xacro"/>
-    <!-- Define Colors -->
-    <material name="white">
-        <color rgba="1 1 1 1"/>
-    </material>
-    <material name="orange">
-        <color rgba="1 0.25 0.1 1"/>
-    </material>
-    <material name="blue">
-        <color rgba="0.2 0.2 1 1"/>
-    </material>
-    <material name="black">
-        <color rgba="0 0 0 1"/>
-    </material>
+    <!-- <xacro:include filename="materials.xacro"/> -->
     <!-- Base Footprint
     <link name="base_footprint"/>
@@ -32,5 +20,5 @@
     <!-- xyz = 172 of box dimesions, x is forward, y is to the sides -->
     <link name="chassis">
-        <visual>
+        <!-- <visual>
             <origin xyz="0.1775 0 0.175" rpy="0 0 0"/>
             <geometry>
@@ -38,5 +26,5 @@
             </geometry>
             <material name="white"/>
-        </visual>
+        </visual> -->
         <collision>
             <origin xyz="0.1775 0 0.175" rpy="0 0 0"/>
@@ -55,5 +43,5 @@
         <parent link="base_link"/>
         <child link="left_wheel"/>
-        <origin xyz="0 0.1865 0" rpy="-${pi/2} 0 0"/>
+        <origin xyz="0 0.188 0" rpy="-${pi/2} 0 0"/>
         <axis xyz="0 0 1"/>
     </joint>
@@ -61,17 +49,17 @@
         <visual>
             <geometry>
-                <cylinder radius="0.044" length="0.01"/>
+                <cylinder radius="0.044" length="0.02"/>
             </geometry>
-            <material name="blue"/>
+            <material name="orange"/>
         </visual>
         <collision>
             <geometry>
-                <cylinder radius="0.044" length="0.01"/>
+                <cylinder radius="0.044" length="0.02"/>
             </geometry>
         </collision>
-        <xacro:inertial_cylinder mass="0.1" length="0.01" radius="0.044"/>
+        <xacro:inertial_cylinder mass="0.1" length="0.02" radius="0.044"/>
     </link>
     <gazebo reference="left_wheel">
-        <material>Gazebo/Blue</material>
+        <material>Gazebo/Orange</material>
     </gazebo>
     <!-- Right Wheel -->
@@ -79,5 +67,5 @@
         <parent link="base_link"/>
         <child link="right_wheel"/>
-        <origin xyz="0 -0.1865 0" rpy="${pi/2} 0 0"/>
+        <origin xyz="0 -0.188 0" rpy="${pi/2} 0 0"/>
         <axis xyz="0 0 -1"/>
     </joint>
@@ -85,17 +73,17 @@
         <visual>
             <geometry>
-                <cylinder radius="0.044" length="0.01"/>
+                <cylinder radius="0.044" length="0.02"/>
             </geometry>
-            <material name="blue"/>
+            <material name="orange"/>
         </visual>
         <collision>
             <geometry>
-                <cylinder radius="0.044" length="0.01"/>
+                <cylinder radius="0.044" length="0.02"/>
             </geometry>
         </collision>
-        <xacro:inertial_cylinder mass="0.1" length="0.01" radius="0.044"/>
+        <xacro:inertial_cylinder mass="0.1" length="0.02" radius="0.044"/>
     </link>
     <gazebo reference="right_wheel">
-        <material>Gazebo/Blue</material>
+        <material>Gazebo/Orange</material>
     </gazebo>
     <!-- Caster Wheel -->
@@ -103,16 +91,16 @@
         <parent link="chassis"/>
         <child link="caster_wheel"/>
-        <origin xyz="0.3 0 0" rpy="0 0 0"/>
+        <origin xyz="-0.11 0 0" rpy="0 0 0"/>
     </joint>
     <link name="caster_wheel">
         <visual>
             <geometry>
-                <sphere radius="0.044"/>
+                <sphere radius="0.02"/>
             </geometry>
-            <material name="black"/>
+            <material name="orange"/>
         </visual>
         <collision>
             <geometry>
-                <sphere radius="0.044"/>
+                <sphere radius="0.02"/>
             </geometry>
             <surface>
@@ -125,8 +113,8 @@
             </surface>
         </collision>
-        <xacro:inertial_sphere mass="0.1" radius="0.044"/>
+        <xacro:inertial_sphere mass="0.1" radius="0.02"/>
     </link>
     <gazebo reference="caster_wheel">
-        <material>Gazebo/Black</material>
+        <material>Gazebo/Orange</material>
         <mu1 value="0.0001"/>
         <mu2 value="0.0001"/>

File: src/robonav/description/rplidar_c1.xacro (robot description, xacro)
@@ -1,4 +1,5 @@
 <?xml version="1.0"?>
 <robot xmlns:xacro="http://www.ros.org/wiki/xacro">
+    <!-- <xacro:include filename="materials.xacro"/> -->
     <!-- Lidar -->
     <link name="lidar_link">
@@ -7,4 +8,5 @@
                 <cylinder radius="0.04" length="0.03"/>
             </geometry>
+            <material name="orange"/>
         </visual>
         <collision>
@@ -25,5 +27,5 @@
         <parent link="base_link"/>
         <child link="lidar_link"/>
-        <origin xyz="-0.053 0.0 0.365" rpy="0 0 0"/>  <!-- Lidar is on top of the Chassis -->
+        <origin xyz="-0.053 0.0 0.36" rpy="0 0 0"/>  <!-- Lidar is on top of the Chassis -->
     </joint>
 </robot>
