Commit message: added start from esp (rpi waits), added colour choosing almost, reset almost from esp, changed speed, wheel diameter

File: src/robonav/description/materials.xacro (robot description, xacro)
@@ -5,5 +5,5 @@
   </material>
   <material name="orange">
-    <color rgba="1 0.25 0.1 1"/>
+    <color rgba="1 0.4 0.2 1"/>
   </material>
   <material name="blue">

File: src/robonav/description/rplidar_c1.xacro (robot description, xacro)
@@ -27,5 +27,5 @@
         <parent link="base_link"/>
         <child link="lidar_link"/>
-        <origin xyz="-0.053 0.0 0.36" rpy="0 0 0"/>  <!-- Lidar is on top of the Chassis -->
+        <origin xyz="-0.053 0.0 0.36" rpy="0 0 3.14159"/>  <!-- Lidar is on top of the Chassis, rotated 180 degrees around the vertical axis -->
     </joint>
 </robot>
