Commit message: Lidar in gazebo working

File: src/robonav/description/rplidar_c1.xacro (robot description, xacro)
@@ -2,5 +2,5 @@
 <robot xmlns:xacro="http://www.ros.org/wiki/xacro">
     <!-- RPLIDAR C1 Sensor -->
-    <link name="rplidar_link">
+    <link name="lidar_link">
         <visual>
             <geometry>
@@ -21,5 +21,5 @@
         </inertial>
     </link>
-    <gazebo reference="rplidar_link">
+    <gazebo reference="lidar_link">
         <material>Gazebo/Black</material>
     </gazebo>
@@ -27,9 +27,10 @@
     <joint name="rplidar_joint" type="fixed">
         <parent link="chassis"/>
-        <child link="rplidar_link"/>
+        <child link="lidar_link"/>
         <origin xyz="0.12 0.0 0.17" rpy="0 0 0"/>  <!-- Lidar sitzt oben auf dem Chassis -->
     </joint>
-    <gazebo reference="rplidar_link">
+    <gazebo reference="lidar_link">
         <sensor type="ray" name="rplidar_sensor">
+            <visualize>true</visualize>
             <update_rate>10</update_rate> <!-- 10 Hz -->
             <ray>
@@ -47,9 +48,17 @@
                     <resolution>0.01</resolution>
                 </range>
+                <noise>
+                    <type>gaussian</type>
+                    <mean>0.0</mean>
+                    <stddev>0.01</stddev>
+                </noise>
             </ray>
-            <plugin name="rplidar_plugin" filename="libgazebo_ros_ray_sensor.so">
-                <topic>scan</topic>
-                <frameName>lidar_frame</frameName>
-                <visualize>true</visualize>
+            <plugin name="lidar_plugin" filename="libgazebo_ros_ray_sensor.so">
+                <ros>
+                <namespace>/</namespace>
+                <remapping>~/out:=scan</remapping>
+                </ros>
+                <output_type>sensor_msgs/LaserScan</output_type>
+                <frame_name>lidar_link</frame_name> <!-- Updated to match the frame name -->
             </plugin>
         </sensor>

Commit message: Lidar specs from C1, added poles in draft.world and ready for lidar programming

File: src/robonav/description/rplidar_c1.xacro (robot description, xacro)
@@ -1,5 +1,5 @@
 <?xml version="1.0"?>
 <robot xmlns:xacro="http://www.ros.org/wiki/xacro">
-    <!-- RPLIDAR C1 Sensor -->
+    <!-- Lidar -->
     <link name="lidar_link">
         <visual>
@@ -24,10 +24,11 @@
         <material>Gazebo/Black</material>
     </gazebo>
-    <!-- Joint zum Roboter (chassis) -->
+    <!-- Joint Lidar to Robot (chassis) -->
     <joint name="rplidar_joint" type="fixed">
         <parent link="chassis"/>
         <child link="lidar_link"/>
-        <origin xyz="0.12 0.0 0.17" rpy="0 0 0"/>  <!-- Lidar sitzt oben auf dem Chassis -->
+        <origin xyz="0.12 0.0 0.35" rpy="0 0 0"/>  <!-- Lidar is on top of the Chassis -->
     </joint>
+    <!-- Lidar Plugin -->
     <gazebo reference="lidar_link">
         <sensor type="ray" name="rplidar_sensor">
@@ -38,5 +39,5 @@
                     <horizontal>
                         <samples>360</samples>
-                        <resolution>1</resolution>
+                        <resolution>0.72</resolution> <!-- Match datasheet -->
                         <min_angle>-3.14159</min_angle>
                         <max_angle>3.14159</max_angle>
@@ -44,12 +45,12 @@
                 </scan>
                 <range>
-                    <min>0.12</min>
+                    <min>0.05</min>
                     <max>12.0</max>
-                    <resolution>0.01</resolution>
+                    <resolution>0.015</resolution>
                 </range>
                 <noise>
                     <type>gaussian</type>
                     <mean>0.0</mean>
-                    <stddev>0.01</stddev>
+                    <stddev>0.015</stddev>  <!-- Noise stddev to match ±30mm accuracy of C1   -->
                 </noise>
             </ray>
@@ -60,5 +61,5 @@
                 </ros>
                 <output_type>sensor_msgs/LaserScan</output_type>
-                <frame_name>lidar_link</frame_name> <!-- Updated to match the frame name -->
+                <frame_name>lidar_link</frame_name>
             </plugin>
         </sensor>

Commit message: Obstacle Detection working, not yet moving, cleaned up files

File: src/robonav/description/rplidar_c1.xacro (robot description, xacro)
@@ -25,5 +25,5 @@
         <parent link="base_link"/>
         <child link="lidar_link"/>
-        <origin xyz="0.1 0.0 0.365" rpy="0 0 0"/>  <!-- Lidar is on top of the Chassis -->
+        <origin xyz="-0.053 0.0 0.365" rpy="0 0 0"/>  <!-- Lidar is on top of the Chassis -->
     </joint>
 </robot>

Commit message: working wiht lidar and my code 1.

File: src/robonav/description/rplidar_c1.xacro (robot description, xacro)
@@ -27,5 +27,5 @@
         <parent link="base_link"/>
         <child link="lidar_link"/>
-        <origin xyz="-0.053 0.0 0.36" rpy="0 0 3.14159"/>  <!-- Lidar is on top of the Chassis, rotated 180 degrees around the vertical axis -->
+        <origin xyz="-0.053 0.0 0.36" rpy="0 0 0.096"/>  <!-- Lidar is on top of the Chassis, rotated 180 degrees around the vertical axis -->
     </joint>
 </robot>
