File: Electrical/Eurobot2025PCB/Eurobot2025PCB.kicad_pcb (KiCad board)
At the start: 2 copper layers, 99 x 99 mm, 25 parts, among them J1 Screw_Terminal_01x02, J2 Conn_01x04_Socket, J3 Conn_01x04_Socket, J4 Conn_01x04_Socket, J5 Conn_01x02_Socket, J6 Conn_01x04_Socket, SW2 SW_SPDT, SW3 SW_Push, SW4 SW_Push, U1 INA219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

Commit message: update pcb :alien:
Parts:
- removed A2: Pololu_Breakout_A4988, ECN:A4988
- removed J2: Conn_01x04_Socket, Connector_JST:JST_XH_B4B-XH-A_1x04_P2.50mm_Vertical
- added REF**: MountingHole_3.2mm_M3, MountingHole:MountingHole_3.2mm_M3, F.Cu at (183.5, 134.5)
- added REF**: D_DO-41_SOD81_P10.16mm_Horizontal, Diode_THT:D_DO-41_SOD81_P10.16mm_Horizontal, F.Cu at (123.0, 131.2)
- added REF**: MountingHole_3.2mm_M3, MountingHole:MountingHole_3.2mm_M3, F.Cu at (96.0, 47.0)
- added REF**: PinSocket_1x04_P2.54mm_Horizontal, Connector_PinSocket_2.54mm:PinSocket_1x04_P2.54mm_Horizontal, F.Cu at (123.4, 57.1)
- added REF**: MountingHole_3.2mm_M3, MountingHole:MountingHole_3.2mm_M3, F.Cu at (183.0, 47.0)
- added REF**: MountingHole_3.2mm_M3, MountingHole:MountingHole_3.2mm_M3, F.Cu at (96.0, 134.5)
- added REF**: Symbol_CC-ShareAlike_CopperTop_Small, Symbol:Symbol_CC-ShareAlike_CopperTop_Small, F.Cu at (98.0, 107.0)
- added REF**: Symbol_CC-ShareAlike_CopperTop_Small, Symbol:Symbol_CC-ShareAlike_CopperTop_Small, B.Cu at (162.0, 111.0)
- moved U7 1.78 mm to (109.5, 128.0)
Connections:
- A1 pad 10: +3V3 -> Net-(A2-SDA)
- A1 pad 11: +3V3 -> Net-(A2-SDA)
- A1 pad 12: +3V3 -> Net-(A2-SDA)
- A1 pad 2: +3V3 -> Net-(A2-SDA)
- A1 pad 9: enable -> Net-(A2-SDA)
- A3 pad 10: +3V3 -> Net-(A2-SDA)
- A3 pad 11: +3V3 -> Net-(A2-SDA)
- A3 pad 12: +3V3 -> Net-(A2-SDA)
- A3 pad 2: +3V3 -> Net-(A2-SDA)
- A3 pad 9: enable -> Net-(A2-SDA)
- A4 pad 1: GND -> Net-(A2-SDA)
- A4 pad 10: +3V3 -> Net-(A2-SDA)
- A4 pad 11: +3V3 -> Net-(A2-SDA)
- A4 pad 12: +3V3 -> Net-(A2-SDA)
- A4 pad 2: +3V3 -> Net-(A2-SDA)
- A4 pad 3: Net-(A4-1B) -> Net-(A2-SDA)
- A4 pad 4: Net-(A4-1A) -> Net-(A2-SDA)
- A4 pad 5: Net-(A4-2A) -> Net-(A2-SDA)
- A4 pad 6: Net-(A4-2B) -> Net-(A2-SDA)
- A4 pad 7: GND -> Net-(A2-SDA)
- A4 pad 9: enable -> Net-(A2-SDA)
- D1 pad 1: GND -> Net-(A2-SDA)
- ESP32 WROOM 32D DEVKIT1 pad 1: +5V -> Net-(A2-SDA)
- ESP32 WROOM 32D DEVKIT1 pad 11: Net-(A2-STEP) -> Net-(A2-SDA)
- ESP32 WROOM 32D DEVKIT1 pad 12: Net-(A2-DIR) -> Net-(A2-SDA)
- ESP32 WROOM 32D DEVKIT1 pad 16: Net-(ESP32 WROOM 32D DEVKIT1-D23) -> Net-(A2-SDA)
- ESP32 WROOM 32D DEVKIT1 pad 18: Net-(ESP32 WROOM 32D DEVKIT1-TX0) -> Net-(A2-SDA)
- ESP32 WROOM 32D DEVKIT1 pad 19: Net-(ESP32 WROOM 32D DEVKIT1-RX0) -> Net-(A2-SDA)
- ESP32 WROOM 32D DEVKIT1 pad 2: GND -> Net-(A2-SDA)
- ESP32 WROOM 32D DEVKIT1 pad 26: button1 -> Net-(A2-SDA)
- ESP32 WROOM 32D DEVKIT1 pad 27: Net-(ESP32 WROOM 32D DEVKIT1-D2) -> Net-(A2-SDA)
- ESP32 WROOM 32D DEVKIT1 pad 29: GND -> Net-(A2-SDA)
- ESP32 WROOM 32D DEVKIT1 pad 3: button2 -> Net-(A2-SDA)
- ESP32 WROOM 32D DEVKIT1 pad 30: +3V3 -> Net-(A2-SDA)
- ESP32 WROOM 32D DEVKIT1 pad 4: enable -> Net-(A2-SDA)
- J5 pad 1: Net-(ESP32 WROOM 32D DEVKIT1-TX0) -> Net-(A2-SDA)
- J5 pad 2: Net-(ESP32 WROOM 32D DEVKIT1-RX0) -> Net-(A2-SDA)
- J6 pad 1: Net-(A4-2B) -> Net-(A2-SDA)
- J6 pad 2: Net-(A4-2A) -> Net-(A2-SDA)
- J6 pad 3: Net-(A4-1A) -> Net-(A2-SDA)
- J6 pad 4: Net-(A4-1B) -> Net-(A2-SDA)
- R1 pad 2: +5V -> Net-(A2-SDA)
- RV1 pad 1: +3V3 -> Net-(A2-SDA)
- RV1 pad 3: GND -> Net-(A2-SDA)
- SW3 pad 1: +3V3 -> Net-(A2-SDA)
- SW3 pad 2: button1 -> Net-(A2-SDA)
- SW4 pad 1: +3V3 -> Net-(A2-SDA)
- SW4 pad 2: button2 -> Net-(A2-SDA)
- U1 pad 1: +3V3 -> Net-(A2-SDA)
- U1 pad 2: GND -> Net-(A2-SDA)
- U1 pad 3: Net-(ESP32 WROOM 32D DEVKIT1-D23) -> Net-(A2-SDA)
- U2 pad 1: +3V3 -> Net-(A2-SDA)
- U2 pad 2: GND -> Net-(A2-SDA)
- U3 pad 1: GND -> Net-(A2-SDA)
- U3 pad 2: Net-(ESP32 WROOM 32D DEVKIT1-D23) -> Net-(A2-SDA)
- U3 pad 4: +5V -> Net-(A2-SDA)
- U4 pad 1: GND -> Net-(A2-SDA)
- U4 pad 2: Net-(ESP32 WROOM 32D DEVKIT1-D2) -> Net-(A2-SDA)
- U4 pad 3: GND -> Net-(A2-SDA)
- U4 pad 4: +5V -> Net-(A2-SDA)
- U4 pad 6: GND -> Net-(A2-SDA)
- U5 pad 1: +3V3 -> Net-(A2-SDA)
- U5 pad 2: GND -> Net-(A2-SDA)
- U5 pad 4: Net-(ESP32 WROOM 32D DEVKIT1-D23) -> Net-(A2-SDA)
- U6 pad 1: +3V3 -> Net-(A2-SDA)
- U6 pad 2: GND -> Net-(A2-SDA)
- U6 pad 4: Net-(ESP32 WROOM 32D DEVKIT1-D23) -> Net-(A2-SDA)
- U7 pad 4: GND -> Net-(A2-SDA)
Routing:
- net Net-(A2-SDA): track 0.00 -> 899.0 mm, vias 0 -> 5
- net +3V3: track 331.1 -> 0.00 mm
- net enable: track 194.1 -> 0.00 mm
- net +5V: track 113.6 -> 6.07 mm, vias 1 -> 0
- net Net-(ESP32 WROOM 32D DEVKIT1-D23): track 61.5 -> 0.00 mm
- net Net-(ESP32 WROOM 32D DEVKIT1-D2): track 46.1 -> 0.00 mm
- net button1: track 35.9 -> 0.00 mm
- net Net-(A2-STEP): track 31.9 -> 0.00 mm
- net Net-(A2-DIR): track 31.5 -> 0.00 mm
- net button2: track 30.9 -> 0.00 mm
- net VCC: track 247.8 -> 266.4 mm
- net Net-(ESP32 WROOM 32D DEVKIT1-RX0): track 16.6 -> 0.00 mm
- net Net-(ESP32 WROOM 32D DEVKIT1-TX0): track 14.1 -> 0.00 mm
- net Net-(A2-1B): track 7.15 -> 0.00 mm
- net Net-(A2-1A): track 7.14 -> 0.00 mm
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Other:
- outline, holes or cut-outs redrawn
- board text added: "VL6180X"

Commit message: updated PCB
Parts:
- removed REF** (x4): MountingHole_3.2mm_M3, MountingHole:MountingHole_3.2mm_M3
- removed REF**: D_DO-41_SOD81_P10.16mm_Horizontal, Diode_THT:D_DO-41_SOD81_P10.16mm_Horizontal
- removed REF**: PinSocket_1x04_P2.54mm_Horizontal, Connector_PinSocket_2.54mm:PinSocket_1x04_P2.54mm_Horizontal
- removed REF** (x2): Symbol_CC-ShareAlike_CopperTop_Small, Symbol:Symbol_CC-ShareAlike_CopperTop_Small
- added D2: 1N5817, Diode_THT:D_DO-41_SOD81_P10.16mm_Horizontal, F.Cu at (122.9, 121.4)
- added H1: MountingHole, MountingHole:MountingHole_3.2mm_M3, F.Cu at (94.7, 45.5)
- added H2: MountingHole, MountingHole:MountingHole_3.2mm_M3, F.Cu at (184.7, 45.5)
- added H3: MountingHole, MountingHole:MountingHole_3.2mm_M3, F.Cu at (184.7, 135.6)
- added H4: MountingHole, MountingHole:MountingHole_3.2mm_M3, F.Cu at (94.7, 135.6)
- added SW1: SW_Push_Dual, Connector_PinHeader_2.54mm:PinHeader_2x02_P2.54mm_Vertical, F.Cu at (126.2, 87.1)
- added SW5: SW_Push, Connector_JST:JST_XH_B2B-XH-A_1x02_P2.50mm_Vertical, F.Cu at (123.2, 57.7)
- added U8: PCF8574, Connector_PinHeader_2.54mm:PinHeader_1x04_P2.54mm_Vertical, F.Cu at (172.7, 87.1)
- U3: footprint Connector_PinHeader_2.54mm:PinHeader_1x04_P2.54mm_Vertical -> Connector_PinHeader_2.54mm:PinHeader_1x05_P2.54mm_Vertical
- moved J5 7.37 mm to (164.3, 87.1)
- moved R1 0.63 mm to (185.4, 71.8)
Connections:
- A1 pad 10: Net-(A2-SDA) -> GND
- A1 pad 11: Net-(A2-SDA) -> GND
- A1 pad 12: Net-(A2-SDA) -> GND
- A1 pad 2: Net-(A2-SDA) -> +3V3
- A1 pad 9: Net-(A2-SDA) -> enable
- A3 pad 10: Net-(A2-SDA) -> GND
- A3 pad 11: Net-(A2-SDA) -> GND
- A3 pad 12: Net-(A2-SDA) -> GND
- A3 pad 2: Net-(A2-SDA) -> +3V3
- A3 pad 9: Net-(A2-SDA) -> enable
- A4 pad 1: Net-(A2-SDA) -> GND
- A4 pad 10: Net-(A2-SDA) -> GND
- A4 pad 11: Net-(A2-SDA) -> GND
- A4 pad 12: Net-(A2-SDA) -> GND
- A4 pad 2: Net-(A2-SDA) -> +3V3
- A4 pad 3: Net-(A2-SDA) -> Net-(A4-1B)
- A4 pad 4: Net-(A2-SDA) -> Net-(A4-1A)
- A4 pad 5: Net-(A2-SDA) -> Net-(A4-2A)
- A4 pad 6: Net-(A2-SDA) -> Net-(A4-2B)
- A4 pad 7: Net-(A2-SDA) -> GND
- A4 pad 9: Net-(A2-SDA) -> enable
- D1 pad 1: Net-(A2-SDA) -> GND
- ESP32 WROOM 32D DEVKIT1 pad 1: Net-(A2-SDA) -> Net-(D2-K)
- ESP32 WROOM 32D DEVKIT1 pad 11: Net-(A2-SDA) -> LimitSwitch2
- ESP32 WROOM 32D DEVKIT1 pad 12: Net-(A2-SDA) -> LimitSwitch1
- ESP32 WROOM 32D DEVKIT1 pad 16: Net-(A2-SDA) -> Net-(ESP32 WROOM 32D DEVKIT1-D23)
- ESP32 WROOM 32D DEVKIT1 pad 18: Net-(A2-SDA) -> Net-(ESP32 WROOM 32D DEVKIT1-TX0)
- ESP32 WROOM 32D DEVKIT1 pad 19: Net-(A2-SDA) -> Net-(ESP32 WROOM 32D DEVKIT1-RX0)
- ESP32 WROOM 32D DEVKIT1 pad 2: Net-(A2-SDA) -> GND
- ESP32 WROOM 32D DEVKIT1 pad 26: Net-(A2-SDA) -> button1
- ESP32 WROOM 32D DEVKIT1 pad 27: Net-(A2-SDA) -> Net-(ESP32 WROOM 32D DEVKIT1-D2)
- ESP32 WROOM 32D DEVKIT1 pad 29: Net-(A2-SDA) -> GND
- ESP32 WROOM 32D DEVKIT1 pad 3: Net-(A2-SDA) -> button2
- ESP32 WROOM 32D DEVKIT1 pad 30: Net-(A2-SDA) -> +3V3
- ESP32 WROOM 32D DEVKIT1 pad 4: Net-(A2-SDA) -> enable
- J5 pad 1: Net-(A2-SDA) -> Net-(ESP32 WROOM 32D DEVKIT1-TX0)
- J5 pad 2: Net-(A2-SDA) -> Net-(ESP32 WROOM 32D DEVKIT1-RX0)
- J6 pad 1: Net-(A2-SDA) -> Net-(A4-2B)
- J6 pad 2: Net-(A2-SDA) -> Net-(A4-2A)
- J6 pad 3: Net-(A2-SDA) -> Net-(A4-1A)
- J6 pad 4: Net-(A2-SDA) -> Net-(A4-1B)
- R1 pad 2: Net-(A2-SDA) -> +5V
- RV1 pad 1: Net-(A2-SDA) -> +3V3
- RV1 pad 3: Net-(A2-SDA) -> GND
- SW2 pad 3: VCC -> Net-(SW2-C)
- SW3 pad 1: Net-(A2-SDA) -> +3V3
- SW3 pad 2: Net-(A2-SDA) -> button1
- SW4 pad 1: Net-(A2-SDA) -> +3V3
- SW4 pad 2: Net-(A2-SDA) -> button2
- U1 pad 1: Net-(A2-SDA) -> +3V3
- U1 pad 2: Net-(A2-SDA) -> GND
- U1 pad 3: Net-(A2-SDA) -> Net-(ESP32 WROOM 32D DEVKIT1-D23)
- U2 pad 1: Net-(A2-SDA) -> +3V3
- U2 pad 2: Net-(A2-SDA) -> GND
- U3 pad 1: Net-(A2-SDA) -> GND
- U3 pad 2: Net-(A2-SDA) -> Net-(ESP32 WROOM 32D DEVKIT1-D23)
- U3 pad 4: Net-(A2-SDA) -> +5V
- U4 pad 1: Net-(A2-SDA) -> GND
- U4 pad 2: Net-(A2-SDA) -> Net-(ESP32 WROOM 32D DEVKIT1-D2)
- U4 pad 3: Net-(A2-SDA) -> GND
- U4 pad 4: Net-(A2-SDA) -> +5V
- U4 pad 6: Net-(A2-SDA) -> GND
- U5 pad 1: Net-(A2-SDA) -> +3V3
- U5 pad 2: Net-(A2-SDA) -> GND
- U5 pad 4: Net-(A2-SDA) -> Net-(ESP32 WROOM 32D DEVKIT1-D23)
- U6 pad 1: Net-(A2-SDA) -> +3V3
- U6 pad 2: Net-(A2-SDA) -> GND
- U6 pad 4: Net-(A2-SDA) -> Net-(ESP32 WROOM 32D DEVKIT1-D23)
- U7 pad 4: Net-(A2-SDA) -> GND
Routing:
- net Net-(A2-SDA): track 899.0 -> 0.00 mm, vias 5 -> 0
- net +3V3: track 0.00 -> 338.0 mm
- net enable: track 0.00 -> 159.4 mm
- net +5V: track 6.07 -> 115.7 mm, vias 0 -> 1
- net Net-(ESP32 WROOM 32D DEVKIT1-D23): track 0.00 -> 86.3 mm, vias 0 -> 1
- net Net-(ESP32 WROOM 32D DEVKIT1-D2): track 0.00 -> 39.0 mm
- net VCC: track 266.4 -> 227.9 mm
- net button1: track 0.00 -> 35.9 mm
- net button2: track 0.00 -> 30.9 mm
- net Net-(ESP32 WROOM 32D DEVKIT1-D22): track 60.9 -> 82.1 mm, vias 0 -> 1
- net Net-(D2-K): track 0.00 -> 13.0 mm
- net Net-(ESP32 WROOM 32D DEVKIT1-RX0): track 0.00 -> 9.40 mm
- net Net-(SW2-C): track 0.00 -> 7.67 mm
- net Net-(A4-1B): track 0.00 -> 7.04 mm
- net Net-(A4-1A): track 0.00 -> 7.03 mm
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Other:
- outline, holes or cut-outs redrawn
- board text added: "Author: Alexis MORICE, Laurène BERNIER"
- board text added: "Control Planel"
- board text added: "E-STOP"
- board text added: "LS1"
- board text added: "LS2"
- board text added: "Version: 2.0"
- board text removed: "Author: Alexis MORICE"
- board text removed: "VL6180X"
- board text removed: "Version: 1.0"
